File: hardware/carrier-board/kicad/ProtoHUD-Carrier.kicad_sch (KiCad schematic)
At the start: 0 parts

Commit message: hardware(carrier): replace USB 2.0 hub with VL817 USB 3.1 4-port hub
Swap the on-board USB2514B (USB 2.0) for a VIA VL817 4-port USB 3.1 Gen1
(5 Gbps) hub with four USB-C downstream receptacles (J40-J43), upstream on
a CM5 USB 3.0 port. The CM5 exposes 2x USB 3.0 + 1x USB 2.0, so:

  - USB3 #0 -> VL817 upstream (SuperSpeed + USB 2.0)
  - USB3 #1 -> RP2354B CDC (now OFF-hub, via SW1) -> frees all 4 hub ports
  - USB2    -> backpack phone uplink (J11)

Generator (populate_sheets.py):
  - new VL817 condensed symbol (USB2 + SS per port, xtal, reset, straps)
  - new USB-C 3.1 receptacle symbol (VBUS/GND/CC/D+-/one SS lane)
  - CM5 symbol gains USB3 SuperSpeed pins + 2nd/3rd USB ports
  - rewrite sh_usb(): per-port CC Rp pull-ups (56k, host/DFP), VBUS PTC off
    +5V, USBLC6 ESD, SS AC-coupling caps at each TX, 25 MHz hub clock
  - SW1 'A' side rerouted from hub to the dedicated CM5 USB port

Docs: CONNECTORS, POWER, BOM, REQUIREMENTS, BLOCK-DIAGRAM, READMEs updated
for the USB 3.1 hub, USB-C downstream ports, and off-hub RP2354B link.

All 11 sheets regenerated; S-expressions balanced and cross-sheet global
nets verified consistent.

Co-Authored-By: Claude Opus 4.8 <noreply@anthropic.com>
Claude-Session: https://claude.ai/code/session_01DgiE5SHRCeyk1gvfvshMGa
Other:
- sheet 10. USB Hub renamed 10. USB 3.1 Hub (VL817)
Changed lines of the file:
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@@
   (sheet (at 185.40 57.40) (size 60 25) (fields_autoplaced)
     (stroke (width 0.1524) (type solid)) (fill (color 0 0 0 0.0000))
-    (property "Sheetname" "10. USB Hub" (at 185.40 56.70 0) (effects (font (size 1.27 1.27)) (justify left bottom)))
+    (property "Sheetname" "10. USB 3.1 Hub (VL817)" (at 185.40 56.70 0) (effects (font (size 1.27 1.27)) (justify left bottom)))
     (property "Sheetfile" "usb.kicad_sch" (at 185.40 83.20 0) (effects (font (size 1.27 1.27)) (justify left top)))
   )
